Commit message: add rvix config file and update Dockerfile

File: urdf/robot.urdf (robot description, URDF)
Before this commit: robot mi_robot, 2 links, 1 joints
Joints:
- removed joint mi_junta_esferica
- added joint spherical_joint: type floating, parent link1, child link2, origin xyz=0 0 0 rpy=0 0 0, axis 0 0 1
